File: src-kicad/stm32_master_bt_bat/stm32_master_bt_bat.kicad_pcb (KiCad board)
At the start: 2 copper layers, 40 x 50 mm, 26 parts, among them J1 Conn_01x02_Male, J2 Conn_01x02_Male, J3 Conn_02x04_Odd_Even, J4 Conn_01x06_Female, Q1 Si2371EDS, SW1 SW_Push, SW2 SW_DIP_x01, U1 STM32F031F6Px, Y1 8M

Commit message: Minor fixes in kicad
Parts:
- added F1: Fuse, smd-2410:smd-2410, F.Cu at (237.2, 113.0)
- added H1: MountingHole_Pad, MountingHole:MountingHole_3.2mm_M3_DIN965_Pad, F.Cu at (199.0, 104.0)
- added H2: MountingHole_Pad, MountingHole:MountingHole_3.2mm_M3_DIN965_Pad, F.Cu at (199.0, 146.0)
- added H3: MountingHole_Pad, MountingHole:MountingHole_3.2mm_M3_DIN965_Pad, F.Cu at (241.0, 104.0)
- added H4: MountingHole_Pad, MountingHole:MountingHole_3.2mm_M3_DIN965_Pad, F.Cu at (241.0, 146.0)
- C10, C9, Q1, R5: moved to F.Cu
- C11, C12: footprint Capacitor_THT:CP_Radial_D5.0mm_P2.50mm -> Capacitor_SMD:CP_Elec_6.3x5.8; moved to F.Cu
- C4, C7: footprint Capacitor_THT:CP_Radial_D5.0mm_P2.50mm -> Capacitor_SMD:C_0805_2012Metric_Pad1.18x1.45mm_HandSolder
- C8: footprint Capacitor_THT:CP_Radial_D5.0mm_P2.50mm -> Capacitor_SMD:CP_Elec_6.3x5.8
- SW1: footprint Button_Switch_SMD:Panasonic_EVQPUJ_EVQPUA -> Button_Switch_THT:SW_PUSH_6mm_H5mm
- moved SW1 28.9 mm to (204.0, 108.0)
- moved C7 22.8 mm to (214.0, 136.0)
- moved C5 20.6 mm to (229.8, 130.1)
- moved Q1 20.5 mm to (233.5, 138.0)
- moved C10 20.4 mm to (227.8, 147.1), turned to 90 degrees
- moved C1 20.4 mm to (203.8, 123.4)
- moved C2 20.4 mm to (203.8, 133.1)
- moved C3 20.4 mm to (214.0, 124.2)
- moved C6 20.4 mm to (214.0, 131.0)
- moved C9 20.4 mm to (223.7, 105.9)
- moved J1 20.4 mm to (225.7, 121.8)
- moved J2 20.4 mm to (235.3, 103.0)
- moved J3 20.4 mm to (224.7, 146.6)
- moved J4 20.4 mm to (227.4, 102.6)
- moved R1 20.4 mm to (214.0, 126.5)
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Connections:
- C4 pad 1: +3V3 -> GND
- C4 pad 2: GND -> +3V3
- J2 pad 2: Net-(J2-Pad2) -> Net-(F1-Pad1)
- SW2 pad 1: Net-(J2-Pad2) -> Net-(F1-Pad2)
Routing:
- net Net-(F1-Pad2): track 0.00 -> 7.23 mm
- net Net-(F1-Pad1): track 0.00 -> 6.94 mm
- net Net-(C3-Pad2): track 26.7 -> 32.6 mm
- net Net-(J2-Pad2): track 4.61 -> 0.00 mm
- net Vcc: track 62.6 -> 59.1 mm
- net Net-(R5-Pad1): track 9.79 -> 13.0 mm, vias 1 -> 2
- net +3V3: track 83.3 -> 81.7 mm, vias 0 -> 3
- net GND: track 2.70 -> 4.18 mm, vias 31 -> 39
- net HM-10_STATE: vias 0 -> 1
Other:
- board size 40 x 50 mm -> 50 x 50 mm

Commit message: update src-kicad directory (all files)
Parts:
- removed SW2: SW_DIP_x01, Button_Switch_SMD:SW_DIP_SPSTx01_Slide_6.7x4.1mm_W8.61mm_P2.54mm_LowProfile
- added J5: Conn_01x03, przelbl1x3:PRZELBL1X3, F.Cu at (133.4, 206.8)
- J1: value Conn_01x02_Male -> Conn_01x03_Male; footprint Connector_PinHeader_2.54mm:PinHeader_1x02_P2.54mm_Vertical -> Connector_PinHeader_2.54mm:PinHeader_1x03_P2.54mm_Vertical
- J4: footprint Connector_PinSocket_2.54mm:PinSocket_1x06_P2.54mm_Horizontal -> Connector_PinSocket_2.54mm:PinSocket_1x06_P2.54mm_Vertical
- Y1: footprint Crystal:Crystal_SMD_HC49-SD_HandSoldering -> Crystal:Crystal_SMD_HC49-SD
- moved C9 143.4 mm to (116.3, 200.9)
- moved SW1 140.9 mm to (107.7, 210.8), turned to 90 degrees
- moved C11 138.3 mm to (121.5, 204.5)
- moved C8 138.2 mm to (135.0, 217.4)
- moved J1 138.1 mm to (125.7, 217.1)
- moved C10 137.9 mm to (127.8, 242.1)
- moved C12 137.9 mm to (133.5, 240.0)
- moved C3 137.9 mm to (114.0, 219.2)
- moved C4 137.9 mm to (129.8, 222.6)
- moved C5 137.9 mm to (129.8, 225.1)
- moved C6 137.9 mm to (114.0, 226.0)
- moved H3 137.9 mm to (141.0, 199.0)
- moved H4 137.9 mm to (141.0, 241.0)
- moved J2 137.9 mm to (135.3, 198.0)
- moved J3 137.9 mm to (124.7, 241.6)
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Connections:
- J4 pad 1: HM-10_STATE -> HM-10-BRK
- J4 pad 2: Vcc -> UART1_TXD
- J4 pad 3: GND -> UART1_RXD
- J4 pad 4: UART1_RXD -> GND
- J4 pad 5: UART1_TXD -> Vcc
- J4 pad 6: HM-10-BRK -> HM-10_STATE
Routing:
- net HM-10_STATE: track 30.1 -> 45.2 mm
- net Vcc: track 59.1 -> 67.7 mm
- net +3V3: track 81.7 -> 88.0 mm
- net UART1_TXD: track 33.7 -> 39.7 mm
- net Net-(C3-Pad2): track 32.6 -> 28.5 mm
- net Net-(F1-Pad2): track 7.23 -> 10.7 mm
- net HM-10-BRK: track 33.8 -> 31.1 mm, vias 0 -> 1
- net Net-(F1-Pad1): track 6.94 -> 9.01 mm
- net UART1_RXD: track 40.0 -> 41.9 mm, vias 2 -> 1
- net Net-(C1-Pad1): track 10.9 -> 9.99 mm
- net Net-(C2-Pad1): track 12.2 -> 11.2 mm
- net GND: vias 39 -> 56
Other:
- board size 50 x 50 mm -> 41 x 51 mm
