File: src-kicad/stm32_slave_bat/stm32_slave_bat.sch (KiCad schematic (older format))
At the start: 26 parts, among them J1 Conn_01x02_Male, J2 Conn_01x02_Male, J3 Conn_02x04_Odd_Even, J4 Conn_01x04_Female, Q1 Si2371EDS, SW1 SW_Push, SW2 SW_DIP_x01, U1 STM32F031F6Px, Y1 8M

Commit message: Minor fixes in kicad
Parts:
- removed C4: 4.7u, Capacitor_THT:CP_Radial_D5.0mm_P2.50mm, symbol Device:CP
- removed C7: 1u, Capacitor_THT:CP_Radial_D5.0mm_P2.50mm, symbol Device:CP
- added C4: 4.7u, Capacitor_SMD:C_0805_2012Metric_Pad1.18x1.45mm_HandSolder, symbol Device:C
- added C7: 1u, Capacitor_SMD:C_0805_2012Metric_Pad1.18x1.45mm_HandSolder, symbol Device:C
- added F1: Fuse, smd-2410:smd-2410, symbol Device:Fuse
- added H1, H2, H3, H4: MountingHole_Pad, MountingHole:MountingHole_3.2mm_M3_DIN965, symbol Mechanical:MountingHole_Pad
- C11, C12, C8: footprint Capacitor_THT:CP_Radial_D5.0mm_P2.50mm -> Capacitor_SMD:CP_Elec_6.3x5.8
- SW1: footprint Button_Switch_SMD:Panasonic_EVQPUJ_EVQPUA -> Button_Switch_THT:SW_PUSH_6mm_H5mm
Connections:
- net +3V3: now also C4.2, C7.1
- net GND: now also C4.1, C7.2, H1.1, H2.1, H3.1, H4.1
- net at J2.2 (Pin_2): now also F1.1; no longer SW2.1
- new net: F1.2, SW2.1
Other:
- moved on the sheet: C1, C10, C11, C12, C2, C3, C5, C6, C8, C9, J1, J2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

Commit message: update src-kicad directory (all files)
Parts:
- removed J1: Conn_01x02_Male, Connector_PinHeader_2.54mm:PinHeader_1x02_P2.54mm_Vertical, symbol Connector:Conn_01x02_Male
- removed SW2: SW_DIP_x01, Button_Switch_SMD:SW_DIP_SPSTx01_Slide_6.7x4.1mm_W8.61mm_P2.54mm_LowProfile, symbol Switch:SW_DIP_x01
- added D1: LED, Diode_SMD:D_0805_2012Metric_Pad1.15x1.40mm_HandSolder, symbol Device:LED
- added J1: Conn_01x03_Male, Connector_PinHeader_2.54mm:PinHeader_1x03_P2.54mm_Vertical, symbol Connector:Conn_01x03_Male
- added J5: Conn_01x03, przelbl1x3:PRZELBL1X3, symbol Connector_Generic:Conn_01x03
- added R6: 0, Resistor_SMD:R_0805_2012Metric_Pad1.20x1.40mm_HandSolder, symbol Device:R
- H1, H2, H3, H4: footprint MountingHole:MountingHole_3.2mm_M3_DIN965 -> MountingHole:MountingHole_3.2mm_M3_DIN965_Pad
- Y1: footprint Crystal:Crystal_SMD_HC49-SD_HandSoldering -> Crystal:Crystal_SMD_HC49-SD
Connections:
- net +3V3: now also J5.2 (Pin_2)
- net GND: now also D1.1 (K), J1.3 (Pin_3)
- net SWCLK: now also J1.2 (Pin_2)
- net SWDIO: now also J1.1 (Pin_1)
- net at U1.17 (PA9): now also R6.2
- net at F1.2: now also J5.1 (Pin_1)
- new net: D1.2 (A), R6.1
Changed lines of the file:
@@
 	5150 3550 5350 3550
-Wire Wire Line
-	5350 4250 5150 4250
 Wire Wire Line
 	5150 4350 5350 4350
@@
 F 0 "Y1" V 3254 4381 50  0000 L CNN
 F 1 "8M" V 3345 4381 50  0000 L CNN
-F 2 "Crystal:Crystal_SMD_HC49-SD_HandSoldering" H 3300 4250 50  0001 C CNN
+F 2 "Crystal:Crystal_SMD_HC49-SD" H 3300 4250 50  0001 C CNN
 F 3 "~" H 3300 4250 50  0001 C CNN
 	1    3300 4250
@@
 Wire Wire Line
 	5350 4550 5150 4550
-$Comp
-L Connector:Conn_01x02_Male J1
-U 1 1 5FF2A3AF
-P 5800 4800
-F 0 "J1" V 5862 4844 50  0000 L CNN
-F 1 "Conn_01x02_Male" V 5953 4844 50  0000 L CNN
-F 2 "Connector_PinHeader_2.54mm:PinHeader_1x02_P2.54mm_Vertical" H 5800 4800 50  0001 C CNN
-F 3 "~" H 5800 4800 50  0001 C CNN
-	1    5800 4800
-	0    1    1    0
-$EndComp
 Text GLabel 5800 5100 3    50   Output ~ 0
 SWDIO
@@
 Wire Wire Line
 	5700 5100 5700 5000
-$Comp
-L Switch:SW_DIP_x01 SW2
-U 1 1 5FF6014A
-P 7650 2850
-F 0 "SW2" H 7650 2583 50  0000 C CNN
-F 1 "SW_DIP_x01" H 7650 2674 50  0000 C CNN
-F 2 "Button_Switch_SMD:SW_DIP_SPSTx01_Slide_6.7x4.1mm_W8.61mm_P2.54mm_LowProfile" H 7650 2850 50  0001 C CNN
-F 3 "~" H 7650 2850 50  0001 C CNN
-	1    7650 2850
-	-1   0    0    1
-$EndComp
-Wire Wire Line
-	7350 2850 7200 2850
 $Comp
 L Device:CP C8
@@
 Wire Wire Line
 	7550 5350 7850 5350
-NoConn ~ 5350 4250
 NoConn ~ 5350 4350
 Wire Wire Line
@@
 F 0 "H1" H 2400 6099 50  0000 L CNN
 F 1 "MountingHole_Pad" H 2400 6008 50  0000 L CNN
-F 2 "MountingHole:MountingHole_3.2mm_M3_DIN965" H 2300 6050 50  0001 C CNN
+F 2 "MountingHole:MountingHole_3.2mm_M3_DIN965_Pad" H 2300 6050 50  0001 C CNN
 F 3 "~" H 2300 6050 50  0001 C CNN
 	1    2300 6050
@@
 F 0 "H2" H 2400 6549 50  0000 L CNN
 F 1 "MountingHole_Pad" H 2400 6458 50  0000 L CNN
-F 2 "MountingHole:MountingHole_3.2mm_M3_DIN965" H 2300 6500 50  0001 C CNN
+F 2 "MountingHole:MountingHole_3.2mm_M3_DIN965_Pad" H 2300 6500 50  0001 C CNN
 F 3 "~" H 2300 6500 50  0001 C CNN
 	1    2300 6500
@@
 F 0 "H3" H 2400 6999 50  0000 L CNN
 F 1 "MountingHole_Pad" H 2400 6908 50  0000 L CNN
-F 2 "MountingHole:MountingHole_3.2mm_M3_DIN965" H 2300 6950 50  0001 C CNN
+F 2 "MountingHole:MountingHole_3.2mm_M3_DIN965_Pad" H 2300 6950 50  0001 C CNN
 F 3 "~" H 2300 6950 50  0001 C CNN
 	1    2300 6950
@@
 F 0 "H4" H 2400 7449 50  0000 L CNN
 F 1 "MountingHole_Pad" H 2400 7358 50  0000 L CNN
-F 2 "MountingHole:MountingHole_3.2mm_M3_DIN965" H 2300 7400 50  0001 C CNN
+F 2 "MountingHole:MountingHole_3.2mm_M3_DIN965_Pad" H 2300 7400 50  0001 C CNN
 F 3 "~" H 2300 7400 50  0001 C CNN
 	1    2300 7400
@@
 	1    0    0    -1
 $EndComp
+$Comp
+L Connector_Generic:Conn_01x03 J5
+U 1 1 5FF7C8B7
+P 7650 3200
+F 0 "J5" V 7522 3380 50  0000 L CNN
+F 1 "Conn_01x03" V 7613 3380 50  0000 L CNN
+F 2 "przelbl1x3:PRZELBL1X3" H 7650 3200 50  0001 C CNN
+F 3 "~" H 7650 3200 50  0001 C CNN
+	1    7650 3200
+	0    1    1    0
+$EndComp
+Wire Wire Line
+	7950 2850 7750 2850
+Wire Wire Line
+	7750 2850 7750 3000
+Wire Wire Line
+	7650 3000 7650 2850
+Wire Wire Line
+	7200 2850 7650 2850
+NoConn ~ 7550 3000
+$Comp
+L Device:R R6
+U 1 1 5FF92CB8
+P 5850 4250
+F 0 "R6" V 5643 4250 50  0000 C CNN
+F 1 "0" V 5734 4250 50  0000 C CNN
+F 2 "Resistor_SMD:R_0805_2012Metric_Pad1.20x1.40mm_HandSolder" V 5780 4250 50  0001 C CNN
+F 3 "~" H 5850 4250 50  0001 C CNN
+	1    5850 4250
+	0    1    1    0
+$EndComp
+$Comp
+L Device:LED D1
+U 1 1 5FF94E49
+P 6200 4250
+F 0 "D1" H 6193 3995 50  0000 C CNN
+F 1 "LED" H 6193 4086 50  0000 C CNN
+F 2 "Diode_SMD:D_0805_2012Metric_Pad1.15x1.40mm_HandSolder" H 6200 4250 50  0001 C CNN
+F 3 "~" H 6200 4250 50  0001 C CNN
+	1    6200 4250
+	-1   0    0    1
+$EndComp
+$Comp
+L power:GND #PWR023
+U 1 1 5FF95C54
+P 6400 4500
+F 0 "#PWR023" H 6400 4250 50  0001 C CNN
+F 1 "GND" H 6405 4327 50  0000 C CNN
+F 2 "" H 6400 4500 50  0001 C CNN
+F 3 "" H 6400 4500 50  0001 C CNN
+	1    6400 4500
+	1    0    0    -1
+$EndComp
+Wire Wire Line
+	5150 4250 5700 4250
+Wire Wire Line
+	6000 4250 6050 4250
+Wire Wire Line
+	6350 4250 6400 4250
+Wire Wire Line
+	6400 4250 6400 4500
+$Comp
+L Connector:Conn_01x03_Male J1
+U 1 1 5FFB9548
+P 5700 4800
+F 0 "J1" V 5762 4944 50  0000 L CNN
+F 1 "Conn_01x03_Male" V 5853 4944 50  0000 L CNN
+F 2 "Connector_PinHeader_2.54mm:PinHeader_1x03_P2.54mm_Vertical" H 5700 4800 50  0001 C CNN
+F 3 "~" H 5700 4800 50  0001 C CNN
+	1    5700 4800
+	0    1    1    0
+$EndComp
+$Comp
+L power:GND #PWR024
+U 1 1 5FFBD365
+P 5600 5100
+F 0 "#PWR024" H 5600 4850 50  0001 C CNN
+F 1 "GND" H 5605 4927 50  0000 C CNN
+F 2 "" H 5600 5100 50  0001 C CNN
+F 3 "" H 5600 5100 50  0001 C CNN
+	1    5600 5100
+	1    0    0    -1
+$EndComp
+Wire Wire Line
+	5600 5100 5600 5000
 $EndSCHEMATC
